File: Box_hw/Box_hw.sch (KiCad schematic (older format))
At the start: 98 parts, among them Q1 2N7002, Q2 MMBT2222, Q3 IRLMS9303, SW1 BUTTON, SW2 BUTTON, SW3 BUTTON, SW4 BUTTON, SW5 SWITCH_H, U1 MOC3061M, U2 BTB600

Commit message: * switch to latest libs * Fix "both sns falling" bug
Parts:
- HOLE1, HOLE2, HOLE3, HOLE4: symbol HOLE_METALLED -> HOLE_METALLED-RESCUE-Box_hw
Changed lines of the file:
@@
 EESchema Schematic File Version 2
+LIBS:Box_hw-rescue
 LIBS:Antennas_kl
 LIBS:Connectors_kl
@@
 Connection ~ 12350 5700
 $Comp
-L HOLE_METALLED HOLE1
+L HOLE_METALLED-RESCUE-Box_hw HOLE1
 U 1 1 5467223B
 P 14250 9100
@@
 $EndComp
 $Comp
-L HOLE_METALLED HOLE2
+L HOLE_METALLED-RESCUE-Box_hw HOLE2
 U 1 1 54672241
 P 14250 9450
@@
 $EndComp
 $Comp
-L HOLE_METALLED HOLE3
+L HOLE_METALLED-RESCUE-Box_hw HOLE3
 U 1 1 54672247
 P 14250 9800
@@
 $EndComp
 $Comp
-L HOLE_METALLED HOLE4
+L HOLE_METALLED-RESCUE-Box_hw HOLE4
 U 1 1 5467224D
 P 14250 10150

Commit message: Release
Parts:
- TP1, TP2: symbol TESTPOINT -> TESTPOINT-RESCUE-Box_hw
- XL6: symbol USB_MINI_B -> USB_MINI_B-RESCUE-Box_hw
Changed lines of the file:
@@
 $EndComp
 $Comp
-L TESTPOINT TP1
+L TESTPOINT-RESCUE-Box_hw TP1
 U 1 1 5265B41D
 P 9500 2400
@@
 $EndComp
 $Comp
-L TESTPOINT TP2
+L TESTPOINT-RESCUE-Box_hw TP2
 U 1 1 5265B423
 P 9500 2500
@@
 USB_DM
 $Comp
-L USB_MINI_B XL6
+L USB_MINI_B-RESCUE-Box_hw XL6
 U 1 1 5466B15C
 P 1500 10250
